Commit message: changed pkg name

File: urdf/exosim.urdf (robot description, URDF)
Before this commit: robot oslsim, 12 links, 11 joints
Links:
- link footL: geometry collision box size=0.0675 0.025 0.2; visual mesh filename=package://exosim/meshes/footL.STL
- link footR: geometry collision box size=0.0675 0.025 0.2; visual mesh filename=package://exosim/meshes/footR.STL
- link pylonL: geometry collision box size=0.1 0.35 0.1; visual mesh filename=package://exosim/meshes/pylonLCollider.STL
- link pylonR: geometry collision box size=0.1 0.35 0.1; visual mesh filename=package://exosim/meshes/pylonRCollider.STL
- link thighL: geometry collision box size=0.15 0.3 0.15; visual mesh filename=package://exosim/meshes/thighL.STL
- link thighR: geometry collision box size=0.15 0.3 0.15; visual mesh filename=package://exosim/meshes/thighR.STL
